File: BAR30-SENSOR/BAR30-SENSOR.kicad_pcb (KiCad board)
At the start: 2 copper layers, 17 x 17 mm, 6 parts, among them J1 Conn_01x04_Male, U1 VREG-MIC5365, U2 MS583730BA

Commit message: update
Parts:
- added R1: R, Resistor_SMD:R_0603_1608Metric, F.Cu at (144.8, 102.4)
- added R2: R, Resistor_SMD:R_0603_1608Metric, F.Cu at (157.7, 100.8)
- C1, C2: footprint BAR30-SENSOR:C0402 -> Capacitor_SMD:C_0603_1608Metric
- D1: value DIODESOD523 -> D; footprint BAR30-SENSOR:SOD523 -> Diode_SMD:D_SOD-523
- moved D1 1.08 mm to (147.3, 95.0), turned to 270 degrees
Routing:
- net 3V3: track 12.4 -> 25.2 mm, vias 0 -> 2
- net SCL: track 9.64 -> 21.0 mm, vias 1 -> 2
- net SDA: track 16.8 -> 22.5 mm
- net Net-(C2-Pad1): track 17.7 -> 19.5 mm
Other:
- board text added: "edgecollective.io/pressure"
- board text removed: "C1"
- board text removed: "C2"
- board text removed: "D1"
