File: BAR30-SENSOR/BAR30-SENSOR.sch (KiCad schematic (older format))
At the start: 6 parts, among them J1 Conn_01x04_Male, U1 VREG-MIC5365, U2 MS583730BA

Commit message: update
Parts:
- removed D1: DIODESOD523, BAR30-SENSOR:SOD523, symbol BAR30-SENSOR-eagle-import:DIODESOD523
- added D1: D, Diode_SMD:D_SOD-523, symbol Device:D
- added R1, R2: R, Resistor_SMD:R_0603_1608Metric, symbol Device:R
- C1, C2: footprint BAR30-SENSOR:C0402 -> Capacitor_SMD:C_0603_1608Metric
Connections:
- net 3V3: now also R1.1, R2.1
- net SCL: now also R2.2
- net SDA: now also R1.2
- net VIN: now also D1.2 (A)
- net at C2.1, U1.1 (VIN), U1.3 (EN): now also D1.1 (K)
Changed lines of the file:
@@
 EESchema Schematic File Version 4
+LIBS:BAR30-SENSOR-cache
 EELAYER 26 0
 EELAYER END
@@
 F 0 "C1" H 5260 2415 59  0000 L BNN
 F 1 "1uF" H 5260 2215 59  0000 L BNN
-F 2 "BAR30-SENSOR:C0402" H 5200 2400 50  0001 C CNN
+F 2 "Capacitor_SMD:C_0603_1608Metric" H 5200 2400 50  0001 C CNN
 F 3 "" H 5200 2400 50  0001 C CNN
 	1    5200 2400
@@
 $EndComp
 $Comp
-L BAR30-SENSOR-eagle-import:DIODESOD523 D1
-U 1 0 BE5F3F048D141E84
-P 2200 2100
-F 0 "D1" H 2300 2119 59  0000 L BNN
-F 1 "DIODESOD523" H 2300 2009 59  0000 L BNN
-F 2 "BAR30-SENSOR:SOD523" H 2200 2100 50  0001 C CNN
-F 3 "" H 2200 2100 50  0001 C CNN
-	1    2200 2100
-	1    0    0    -1
-$EndComp
-$Comp
 L BAR30-SENSOR-eagle-import:FRAME-BLUEROBOTICS #FRAME1
 U 1 0 FD5C1A03D2C66578
@@
 F 0 "C2" H 2860 2415 59  0000 L BNN
 F 1 "1uF" H 2860 2215 59  0000 L BNN
-F 2 "BAR30-SENSOR:C0402" H 2800 2400 50  0001 C CNN
+F 2 "Capacitor_SMD:C_0603_1608Metric" H 2800 2400 50  0001 C CNN
 F 3 "" H 2800 2400 50  0001 C CNN
 	1    2800 2400
@@
 SDA
 Wire Wire Line
-	2300 2100 2800 2100
-Wire Wire Line
 	2800 2100 3300 2100
-Connection ~ 2800 2100
 Connection ~ 3300 2100
 Wire Wire Line
@@
 Text GLabel 1900 2100 0    50   Input ~ 0
 VIN
-Wire Wire Line
-	2100 2100 1900 2100
+$Comp
+L Device:R R1
+U 1 1 5CEADC2F
+P 6250 3650
+F 0 "R1" H 6320 3696 50  0000 L CNN
+F 1 "R" H 6320 3605 50  0000 L CNN
+F 2 "Resistor_SMD:R_0603_1608Metric" V 6180 3650 50  0001 C CNN
+F 3 "~" H 6250 3650 50  0001 C CNN
+	1    6250 3650
+	0    1    1    0
+$EndComp
+Text GLabel 6400 3650 2    50   Input ~ 0
+3V3
+Text GLabel 6100 3650 0    50   Input ~ 0
+SDA
+$Comp
+L Device:R R2
+U 1 1 5CEAE4D9
+P 6250 4000
+F 0 "R2" H 6320 4046 50  0000 L CNN
+F 1 "R" H 6320 3955 50  0000 L CNN
+F 2 "Resistor_SMD:R_0603_1608Metric" V 6180 4000 50  0001 C CNN
+F 3 "~" H 6250 4000 50  0001 C CNN
+	1    6250 4000
+	0    1    1    0
+$EndComp
+Text GLabel 6400 4000 2    50   Input ~ 0
+3V3
+Text GLabel 6100 4000 0    50   Input ~ 0
+SCL
+$Comp
+L Device:D D1
+U 1 1 5CEB6F87
+P 2300 2100
+F 0 "D1" H 2300 1884 50  0000 C CNN
+F 1 "D" H 2300 1975 50  0000 C CNN
+F 2 "Diode_SMD:D_SOD-523" H 2300 2100 50  0001 C CNN
+F 3 "~" H 2300 2100 50  0001 C CNN
+	1    2300 2100
+	-1   0    0    1
+$EndComp
+Wire Wire Line
+	2150 2100 1900 2100
+Wire Wire Line
+	2450 2100 2800 2100
+Connection ~ 2800 2100
 $EndSCHEMATC
