File: through-simple/BAR30-SENSOR.kicad_pcb (KiCad board)
At the start: 2 copper layers, 64 x 30 mm, 4 parts, among them J1 Conn_01x04_Male, J2 Conn_01x04_Male, U2 MS583730BA

Commit message: update
Parts:
- moved J2 42.1 mm to (92.6, 53.2)
- moved C1 42.1 mm to (55.8, 44.1)
- moved J1 42.1 mm to (58.6, 53.2)
- moved U2 42.1 mm to (54.8, 48.4)
Other:
- board size 64 x 30 mm -> 67 x 33 mm
- board text added: "edgecollective.io/cuttle"
- board text removed: "U1"
- board text removed: "U2"
- board text removed: "VIN"
- board text removed: "edgecollective.io/pressure"
