File: through-square/BAR30-SENSOR.kicad_pcb (KiCad board)
At the start: 2 copper layers, 33 x 33 mm, 3 parts, among them J1 Conn_01x04_Male, U2 MS583730BA

Commit message: update
Other:
- board size 33 x 33 mm -> 32.9 x 32.9 mm
Changed lines of the file:
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@@
   (general
     (thickness 1.6)
-    (drawings 7)
+    (drawings 14)
     (tracks 19)
     (zones 0)
@@
   )
   (setup
-    (last_trace_width 1.4)
+    (last_trace_width 0.25)
     (user_trace_width 0.35)
     (user_trace_width 1.1)
@@
     )
   )
+  (gr_line (start 42.3 32.4) (end 54.9 26.7) (layer Edge.Cuts) (width 0.15))
+  (gr_line (start 38.3 43.7) (end 42.3 32.4) (layer Edge.Cuts) (width 0.15))
+  (gr_line (start 43.5 55.1) (end 38.3 43.7) (layer Edge.Cuts) (width 0.15))
+  (gr_line (start 54.8 59.6) (end 43.5 55.1) (layer Edge.Cuts) (width 0.15))
+  (gr_line (start 65.9 55.3) (end 54.8 59.6) (layer Edge.Cuts) (width 0.15))
+  (gr_line (start 71.2 43.7) (end 65.9 55.3) (layer Edge.Cuts) (width 0.15))
+  (gr_line (start 67.4 32.5) (end 71.2 43.7) (layer Edge.Cuts) (width 0.15))
+  (gr_line (start 54.9 26.7) (end 67.4 32.5) (layer Edge.Cuts) (width 0.15))
   (gr_line (start 54.82336 53.28936) (end 54.82336 59.63936) (layer Dwgs.User) (width 0.15))
-  (gr_circle (center 54.82336 43.13936) (end 71.32336 43.13936) (layer Edge.Cuts) (width 0.15))
   (gr_text edgecollective.io/cuttle (at 55.118 37.29736) (layer F.SilkS)
     (effects (font (size 1 1) (thickness 0.15)))
